File: Boards/Reflow Skillet Rev 1/Reflow Skillet Rev 1.kicad_pcb (KiCad board)
At the start: 2 copper layers, 78 x 44 mm, 14 parts, among them J1 Output, SW1 Start/Stop, SW2 Pause

Commit message: As sent to jlcpcb
Parts:
- added G***: LOGO, MyFlamingoLogo:flamingo_logo_26_20_mm, B.Cu at (132.1, 48.3)
- turned R1 to 180 degrees
Routing:
- net VBUS: track 0.00 -> 111.6 mm
- net Net-(U1-SDI): track 0.00 -> 74.7 mm, vias 0 -> 2
- net Net-(U1-SCK): track 0.00 -> 68.2 mm, vias 0 -> 4
- net Net-(U2-8): track 0.00 -> 65.6 mm, vias 0 -> 4
- net Net-(U2-6~): track 0.00 -> 58.9 mm, vias 0 -> 2
- net Net-(U2-5~): track 0.00 -> 58.3 mm, vias 0 -> 2
- net Net-(U2-3~): track 0.00 -> 52.8 mm
- net Net-(U2-4): track 0.00 -> 42.9 mm
- net Net-(U1-SDO): track 0.00 -> 22.5 mm, vias 0 -> 2
- net Net-(U1-FAULT): track 0.00 -> 11.6 mm, vias 0 -> 2
- net Net-(U1-CS): track 0.00 -> 10.0 mm
- net Net-(U1-DRDY): track 0.00 -> 8.49 mm, vias 0 -> 2
- net Net-(J1-Pin_2): track 0.00 -> 8.43 mm
- net GND: vias 0 -> 14
- added copper zone on B.Cu, net GND
- added copper zone on F.Cu, net GND
